Commit message: Dataset para roboflow

File: ros2_ws/src/wind_tower_description/urdf/inspection_camera_lighting.urdf.xacro (robot description, xacro)
@@ -53,5 +53,6 @@
     <parent link="inspection_camera_lens_link"/>
     <child link="inspection_camera_optical_frame"/>
-    <origin xyz="0.06 0 0" rpy="0 0 0"/>
+    <!-- ROS optical frame: Z forward along the lens, X right, Y down. -->
+    <origin xyz="0.06 0 0" rpy="-1.5708 0 -1.5708"/>
   </joint>
   <link name="inspection_light_left_link">

Commit message: Lo que me quedo de mi rama y arreglo test YOLO (Ya va)

File: ros2_ws/src/wind_tower_description/urdf/inspection_camera_lighting.urdf.xacro (robot description, xacro)
@@ -53,6 +53,5 @@
     <parent link="inspection_camera_lens_link"/>
     <child link="inspection_camera_optical_frame"/>
-    <!-- ROS optical frame: Z forward along the lens, X right, Y down. -->
-    <origin xyz="0.06 0 0" rpy="-1.5708 0 -1.5708"/>
+    <origin xyz="0.06 0 0" rpy="0 0 0"/>
   </joint>
   <link name="inspection_light_left_link">
